File: Hw 2.X/HW2&3/schematic.brd (EAGLE design)
At the start: 160 x 100 mm, 23 parts, among them J1 USB-MB-H

Commit message: Made Board
Parts:
- moved R2 96.6 mm to (96.8, 71.5), turned to 180 degrees
- moved LED2 85.3 mm to (85.6, 71.5)
- moved R4 50.7 mm to (73.6, 78.2)
- moved R1 25.6 mm to (145.5, 65.9)
- moved LED1 25.0 mm to (134.3, 66.1)
- moved C3 12.7 mm to (75.0, 63.7)
- moved VCAP 7.79 mm to (65.2, 53.8), turned to 180 degrees
- moved RESET 0.63 mm to (92.3, 24.2)
- moved USER 0.54 mm to (84.8, 78.2)
- moved R3 0.17 mm to (46.8, 10.9)
- moved C4 0.13 mm to (29.7, 2.77)
Routing:
- net +3V3: track 0.00 -> 274.6 mm, vias 0 -> 14
- net +5V: track 0.00 -> 152.7 mm, vias 0 -> 3
- net ID: track 0.00 -> 139.7 mm, vias 0 -> 3
- net D+: track 0.00 -> 116.4 mm, vias 0 -> 4
- net D-: track 0.00 -> 108.6 mm, vias 0 -> 2
- net B4/USER: track 0.00 -> 104.4 mm, vias 0 -> 3
- net A4/LED: track 0.00 -> 92.0 mm, vias 0 -> 3
- net MCLR: track 0.00 -> 85.1 mm, vias 0 -> 3
- net A0: track 0.00 -> 84.5 mm, vias 0 -> 2
- net A1: track 0.00 -> 80.5 mm, vias 0 -> 2
- net B15: track 0.00 -> 77.1 mm, vias 0 -> 2
- net B2: track 0.00 -> 76.6 mm, vias 0 -> 2
- net B7: track 0.00 -> 74.7 mm, vias 0 -> 4
- net B3: track 0.00 -> 74.5 mm
- net B8: track 0.00 -> 72.9 mm, vias 0 -> 2
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
Commit message: adjust board
Routing:
- net B7: track 74.7 -> 75.0 mm, vias 4 -> 3
Changed lines of the file:
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@@
 <wire x1="71.4502" y1="62.0776" x2="73.0504" y2="62.0776" width="0.254" layer="1"/>
 <via x="73.0504" y="62.0776" extent="1-16" drill="0.35"/>
-<wire x1="73.0504" y1="62.0776" x2="73.0504" y2="60.4604" width="0.254" layer="16"/>
-<wire x1="73.0504" y1="60.4604" x2="73" y2="60.41" width="0.254" layer="16"/>
-<via x="73" y="60.41" extent="1-16" drill="0.35"/>
+<wire x1="73.0504" y1="62.0776" x2="73.152" y2="61.976" width="0.254" layer="16"/>
+<wire x1="73.152" y1="60.562" x2="73" y2="60.41" width="0.254" layer="16"/>
+<wire x1="73.0504" y1="62.0776" x2="73" y2="62.0272" width="0.1524" layer="1"/>
+<wire x1="73" y1="62.0272" x2="73" y2="60.41" width="0.1524" layer="1"/>
+<wire x1="73" y1="60.41" x2="73" y2="60.41" width="0" layer="19" extent="1-16"/>
 </signal>
 <signal name="B8">
